File: FrontEnd/Common/NoiseSource/NoiseSource.kicad_pcb (KiCad board)
At the start: 2 copper layers, 94 x 30 mm, 286 parts, among them P1 BNC, U1 PMA-545G1_Amp, U2 PMA-545G1_Amp, U3 PMA-545G1_Amp, U4 HSWA2-30DR_switch, U5 HSWA2-30DR_switch, U6 HSWA2-30DR_switch, U7 SN74LVC2G17_Schmitt, U8 SN74LVC2G17_Schmitt, U9 SN74LVC2GU04_Invert

Commit message: [Added] More parts
Parts:
- removed the ? at (160.6, 78.7)
- removed the ? at (160.5, 68.0)
- removed the ? at (134.3, 68.1)
- removed the ? at (134.4, 78.8)
- added ?: , Minicircuits:30mil-30mil_90_Arc, F.Cu at (136.6, 78.0)
- added ?: , Minicircuits:30mil-30mil_90_Arc, F.Cu at (136.6, 69.7)
- added ?: , Minicircuits:30mil-30mil_90_Arc, F.Cu at (158.3, 69.7)
- added ?: , Minicircuits:30mil-30mil_90_Arc, F.Cu at (158.3, 78.0)
- added C19: 0.1Uf, Capacitors_SMD:C_0603, F.Cu at (153.6, 73.8)
- added C20: 0.1Uf, Capacitors_SMD:C_0603, F.Cu at (140.8, 71.4)
- added C21: 0.1Uf, Capacitors_SMD:C_0603, F.Cu at (175.7, 67.1)
- added C22: 0.1Uf, Capacitors_SMD:C_0603, F.Cu at (139.8, 59.9)
- added U10: SN74AUP1T86_Schmitt_XOR, DigitalLogic:TI_DCK, F.Cu at (175.9, 73.7)
- U7, U8: value SN74LVC2G17_Schmitt -> SN74AUP1T86_Schmitt_XOR; footprint DigitalLogic:SN74LVC2G17_Schmitt -> DigitalLogic:TI_DCK
- U9: value SN74LVC2GU04_Invert -> SN74AUP1T86_Schmitt_XOR; footprint DigitalLogic:SN74LVC2G17_Schmitt -> DigitalLogic:TI_DCK
- moved U9 46.6 mm to (175.9, 69.6), turned to 180 degrees
- moved U7 33.0 mm to (143.8, 62.6), turned to 270 degrees
- moved U8 8.96 mm to (143.8, 60.1)
- moved C11 2.93 mm to (120.2, 82.3)
- moved C5 2.92 mm to (104.0, 82.3)
- moved ? 1.50 mm to (141.2, 79.1)
- moved ? 1.50 mm to (141.2, 78.4)
- moved ? 1.50 mm to (140.5, 79.2)
- moved ? 1.50 mm to (140.5, 78.4)
- moved ? 1.50 mm to (144.2, 81.3)
- moved ? 1.50 mm to (144.6, 80.1)
- moved ? 1.50 mm to (145.3, 80.2)
- moved ? 1.50 mm to (145.4, 79.2)
- moved ? 1.50 mm to (143.6, 80.2)
- moved ? 1.50 mm to (143.2, 86.7)
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Connections:
- ? pad 1: Net-(C6-Pad2) -> Net-(C12-Pad2)
- U7 pad 1: Net-(U7-Pad1) -> +3V3
- U7 pad 2: GND -> SolarSel
- U7 pad 3: ShuntSel -> GND
- U7 pad 4: ShuntCTRL1 -> CTRL1
- U7 pad 5: +3V3 -> Net-(U7-Pad5)
- U7 pad 6: ShuntCTRL2 -> +3V3
- U8 pad 1: Net-(U8-Pad1) -> SolarSel
- U8 pad 3: SolarSel -> GND
- U8 pad 5: +3V3 -> Net-(U8-Pad5)
- U8 pad 6: CTRL1 -> +3V3
- U9 pad 1: ShuntSel -> +3V3
- U9 pad 2: GND -> ShuntSel
- U9 pad 3: SolarSel -> GND
- U9 pad 4: Net-(U8-Pad1) -> ShuntCTRL1
- U9 pad 5: +3V3 -> Net-(U9-Pad5)
- U9 pad 6: Net-(U7-Pad1) -> +3V3
Routing:
- net +3V3: track 0.00 -> 74.3 mm, vias 0 -> 2
- net ShuntSel: track 0.00 -> 54.1 mm
- net +5V: track 25.7 -> 57.6 mm
- net SolarSel: track 0.00 -> 8.52 mm, vias 0 -> 3
- net ShuntCTRL1: track 0.00 -> 7.91 mm
- net CTRL2: track 15.0 -> 21.7 mm
- net Net-(U4-Pad3): track 28.9 -> 22.6 mm
- net ShuntCTRL2: track 0.00 -> 5.26 mm
- net CTRL1: track 8.21 -> 11.9 mm
- net Net-(C13-Pad2): track 6.40 -> 4.17 mm
- net Net-(C18-Pad1): track 6.05 -> 3.83 mm
- net TVDD: track 17.9 -> 19.7 mm
- net TCTRL2: track 15.4 -> 16.5 mm
- net TCTRL1: track 20.5 -> 21.6 mm
- net Net-(C6-Pad2): track 8.32 -> 7.34 mm
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Other:
- board size 94 x 30 mm -> 93.5 x 34.8 mm
