File: Control/SiteControl/SiteControl.kicad_pcb (KiCad board)
At the start: 2 copper layers, 52.5 x 115.5 mm, 162 parts, among them J1 RJ50, J2 CONN_01X03, J3 IDC_16Pin_Polarized, J4 CONN_01X06, J5 IDC-10_Polarized, J6 CONN_01X02, J7 Molex Minifit-JR 4.2mm, Q1 BC817-40, Q2 SI2323DDS-T1-GE3, U1 Opto_H11L1M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

Commit message: [Added] Test Pads to Site Control Board; [Completed] Site contorl board DRC
Parts:
- added ?: , DigitalLogic:Via, F.Cu at (194.5, 134.9)
- added ?: , DigitalLogic:Via, F.Cu at (189.5, 101.4)
- added ?: , DigitalLogic:Via, F.Cu at (186.2, 67.5)
- added ?: , DigitalLogic:Via, F.Cu at (185.6, 75.6)
- added ?: , DigitalLogic:Via, F.Cu at (158.3, 73.2)
- added ?: , DigitalLogic:Via, F.Cu at (173.0, 74.5)
- added ?: , DigitalLogic:Via, F.Cu at (172.8, 68.7)
- added ?: , DigitalLogic:Via, F.Cu at (151.4, 100.6)
- added ?: , DigitalLogic:Via, F.Cu at (156.2, 89.2)
- added ?: , DigitalLogic:Via, F.Cu at (178.0, 132.5)
- added ?: , DigitalLogic:Via, F.Cu at (188.0, 132.8)
- added ?: , DigitalLogic:Via, F.Cu at (190.9, 134.8)
- added ?: , DigitalLogic:Via, F.Cu at (184.1, 132.9)
- added ?: , DigitalLogic:Via, F.Cu at (180.8, 133.0)
- added ?: , DigitalLogic:Via, F.Cu at (199.4, 134.6)
- added ?: , DigitalLogic:Via, F.Cu at (199.2, 138.4)
- added ?: , DigitalLogic:Via, F.Cu at (199.2, 143.2)
- added ?: , DigitalLogic:Via, F.Cu at (199.4, 147.4)
- added ?: , DigitalLogic:Via, F.Cu at (153.3, 132.9)
- added ?: , DigitalLogic:Via, F.Cu at (158.4, 132.9)
- added ?: , DigitalLogic:Via, F.Cu at (152.5, 144.9)
- added ?: , DigitalLogic:Via, F.Cu at (152.1, 149.8)
- added ?: , DigitalLogic:Via, F.Cu at (187.6, 134.9)
- added ?: , DigitalLogic:Via, F.Cu at (152.2, 153.6)
- added ?: , DigitalLogic:Via, F.Cu at (155.2, 155.3)
- added ?: , DigitalLogic:Via, F.Cu at (160.0, 155.3)
- added ?: , DigitalLogic:Via, F.Cu at (174.1, 148.2)
- added ?: , DigitalLogic:Via, F.Cu at (176.6, 148.3)
- added ?: , DigitalLogic:Via, F.Cu at (185.8, 146.1)
- added ?: , DigitalLogic:Via, F.Cu at (183.0, 146.2)
- added ?: , DigitalLogic:Via, F.Cu at (180.4, 146.3)
- added ?: , DigitalLogic:Via, F.Cu at (199.7, 44.8)
- added ?: , DigitalLogic:Via, F.Cu at (196.4, 44.8)
- added ?: , DigitalLogic:Via, F.Cu at (185.4, 135.0)
- added ?: , DigitalLogic:Via, F.Cu at (197.4, 68.3)
- added ?: , DigitalLogic:Via, F.Cu at (200.1, 69.9)
- added ?: , DigitalLogic:Via, F.Cu at (200.2, 74.7)
- added ?: , DigitalLogic:Via, F.Cu at (200.2, 78.4)
- added ?: , DigitalLogic:Via, F.Cu at (200.2, 81.7)
- added ?: , DigitalLogic:Via, F.Cu at (200.2, 84.5)
- added ?: , DigitalLogic:Via, F.Cu at (200.2, 87.0)
- added ?: , DigitalLogic:Via, F.Cu at (177.9, 94.9)
- added ?: , DigitalLogic:Via, F.Cu at (178.4, 92.5)
- added ?: , DigitalLogic:Via, F.Cu at (181.3, 92.9)
- added ?: , DigitalLogic:Via, F.Cu at (186.9, 144.0)
- added ?: , DigitalLogic:Via, F.Cu at (181.4, 90.8)
- added ?: , DigitalLogic:Via, F.Cu at (184.8, 90.8)
- added ?: , DigitalLogic:Via, F.Cu at (188.5, 90.7)
- added ?: , DigitalLogic:Via, F.Cu at (187.6, 94.2)
- added ?: , DigitalLogic:Via, F.Cu at (189.5, 94.1)
- added ?: , DigitalLogic:Via, F.Cu at (185.9, 94.1)
- added ?: , DigitalLogic:Via, F.Cu at (200.2, 89.1)
- added ?: , DigitalLogic:Via, F.Cu at (200.2, 91.8)
- added ?: , DigitalLogic:Via, F.Cu at (152.0, 90.4)
- added ?: , DigitalLogic:Via, F.Cu at (152.0, 88.8)
- added ?: , DigitalLogic:Via, F.Cu at (183.3, 144.0)
- added ?: , Measurement_Points:Measurement_Point_Round-SMD-Pad_Small, B.Cu at (196.9, 105.0)
- added ?: , Measurement_Points:Measurement_Point_Round-SMD-Pad_Small, B.Cu at (168.6, 71.5)
- added ?: , Measurement_Points:Measurement_Point_Round-SMD-Pad_Small, B.Cu at (185.9, 115.2)
- added ?: , Measurement_Points:Measurement_Point_Round-SMD-Pad_Small, B.Cu at (164.6, 133.0)
- added ?: , Measurement_Points:Measurement_Point_Round-SMD-Pad_Small, B.Cu at (158.1, 130.2)
- added ?: , Measurement_Points:Measurement_Point_Round-SMD-Pad_Small, B.Cu at (153.6, 130.2)
- added ?: , Measurement_Points:Measurement_Point_Round-SMD-Pad_Small, B.Cu at (151.4, 130.2)
- added ?: , Measurement_Points:Measurement_Point_Round-SMD-Pad_Small, B.Cu at (155.9, 130.2)
- added ?: , Measurement_Points:Measurement_Point_Round-SMD-Pad_Small, B.Cu at (198.1, 72.2)
- added ?: , Measurement_Points:Measurement_Point_Round-SMD-Pad_Small, F.Cu at (194.4, 81.5)
- added ?: , DigitalLogic:Via, F.Cu at (191.4, 101.5)
- added ?: , Measurement_Points:Measurement_Point_Round-SMD-Pad_Small, B.Cu at (183.9, 74.8)
- added ?: , Measurement_Points:Measurement_Point_Round-SMD-Pad_Small, B.Cu at (184.9, 77.8)
- added ?: , Measurement_Points:Measurement_Point_Round-SMD-Pad_Small, B.Cu at (190.9, 79.2)
- added ?: , Measurement_Points:Measurement_Point_Round-SMD-Pad_Small, B.Cu at (160.4, 70.5)
- added ?: , Measurement_Points:Measurement_Point_Round-SMD-Pad_Small, B.Cu at (186.4, 82.5)
- added ?: , Measurement_Points:Measurement_Point_Round-SMD-Pad_Small, F.Cu at (175.1, 153.8)
- added ?: , Measurement_Points:Measurement_Point_Round-SMD-Pad_Small, F.Cu at (169.4, 115.5)
- added ?: , DigitalLogic:Via, F.Cu at (191.5, 103.3)
- added ?: , Measurement_Points:Measurement_Point_Round-SMD-Pad_Small, F.Cu at (196.9, 105.0)
- added ?: , DigitalLogic:Via, F.Cu at (189.4, 103.5)
- moved VR1 0.45 mm to (193.9, 126.0)
Routing:
- net RPi_En: track 84.7 -> 93.3 mm
- net RPi_5V_En: track 110.7 -> 117.0 mm
- net RTC_nCS: track 42.2 -> 47.7 mm
- net GND: track 943.5 -> 948.9 mm
- net RPi_5V_PGood: track 104.9 -> 108.6 mm
- net Modem_En: track 66.9 -> 70.0 mm
- net ADC_nCS: track 59.6 -> 62.2 mm
- net Net-(J7-Pad2): track 4.35 -> 2.03 mm
- net Net-(P1-Pad2): track 6.26 -> 8.58 mm
- net SDI: track 71.2 -> 72.6 mm, vias 4 -> 5
- net SCLK: track 69.8 -> 71.1 mm
- net SDO: track 70.1 -> 71.1 mm
Other:
- board text added: "+3V3"
- board text added: "+5V"
- board text added: "+BATT"
- board text added: "5VE"
- board text added: "5VG"
- board text added: "A_CS"
- board text added: "GND"
- board text added: "MEn"
- board text added: "PiE"
- board text added: "R_CS"
- board text added: "SCLK"
- board text added: "SDI"
- board text added: "SDO"

Commit message: [Updated] RF Modem power port to include an additional ground wire; [Fixed] LM43602 footprint vias by increasing their drill size to 13mils
Parts:
- J6: value CONN_01X02 -> CONN_01X03; footprint Terminal_Blocks:TerminalBlock_Pheonix_MPT-2.54mm_2pol -> Terminal_Blocks:TerminalBlock_Pheonix_MPT-2.54mm_3pol
Connections:
- J7 pad 2: Net-(P1-Pad2) -> Net-(J7-Pad2)
Routing:
- net Net-(P1-Pad2): track 8.58 -> 0.00 mm
- net Net-(J7-Pad2): track 2.03 -> 10.6 mm
- net RPi_5V_En: track 117.0 -> 116.1 mm
Other:
- board text added: "VM+ VM- GND"
- board text removed: "VM+ VM-"
